File: elec/layout/default/femtofox-mppt.kicad_pcb (KiCad board)
At the start: 2 copper layers, 40 x 40 mm, 0 parts

Commit message: checkpoint
Parts:
- added C1: 10V 100nF X5R ±10% 0201 Multilayer Ceramic Capacitors MLCC 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, lib:C0201, F.Cu at (212.3, 50.3)
- added C10: 10V 10uF X5R ±10% 0603 Multilayer Ceramic Capacitors MLCC -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, lib:C0603, F.Cu at (209.7, 72.4)
- added C11: 10V 10uF X5R ±10% 0603 Multilayer Ceramic Capacitors MLCC -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, lib:C0603, F.Cu at (210.9, 66.9)
- added C12: 10V 10uF X5R ±10% 0603 Multilayer Ceramic Capacitors MLCC -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, lib:C0603, F.Cu at (215.7, 72.4)
- added C2: 25V 1uF X5R ±10% 0402 Multilayer Ceramic Capacitors MLCC - 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, lib:C0402, F.Cu at (203.1, 82.0)
- added C3: 6.3V 10uF X5R ±20% 0402 Multilayer Ceramic Capacitors MLCC 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, lib:C0402, F.Cu at (203.1, 85.9)
- added C4: 10V 4.7uF X5R ±20% 0402 Multilayer Ceramic Capacitors MLCC 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, lib:C0402, F.Cu at (208.5, 84.6)
- added C5: 50V 47nF X7R ±10% 0402 Multilayer Ceramic Capacitors MLCC -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, lib:C0402, F.Cu at (208.5, 80.6)
- added C6: 6.3V 10uF X5R ±20% 0402 Multilayer Ceramic Capacitors MLCC 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, lib:C0402, F.Cu at (208.5, 76.7)
- added C7: 6.3V 10uF X5R ±20% 0402 Multilayer Ceramic Capacitors MLCC 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, lib:C0402, F.Cu at (213.4, 80.6)
- added C8: 6.3V 10uF X5R ±20% 0402 Multilayer Ceramic Capacitors MLCC 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, lib:C0402, F.Cu at (213.4, 76.7)
- added C9: 6.3V 22uF X5R ±20% 0603 Multilayer Ceramic Capacitors MLCC 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, lib:C0603, F.Cu at (203.7, 72.4)
- added J1: ?, lib:CONN-SMD_4P-P1.00_SM04B-SRSS-TB-LF-SN, F.Cu at (196.8, 99.9)
- added R1: 50mW Thick Film Resistors 25V ±1% ±200ppm/℃ 120Ω 0201 Chip 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, lib:R0201, F.Cu at (216.7, 50.3)
- added R10: 50mW Thick Film Resistors 25V ±1% ±200ppm/℃ 10kΩ 0201 Chip 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, lib:R0201, F.Cu at (212.3, 57.8)
- added R11: 50mW Thick Film Resistors 25V ±1% ±200ppm/℃ 10kΩ 0201 Chip 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, lib:R0201, F.Cu at (212.3, 54.1)
- added R12: 50mW Thick Film Resistors 25V ±1% ±200ppm/℃ 10kΩ 0201 Chip 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, lib:R0201, F.Cu at (216.7, 57.8)
- added R2: 50mW Thick Film Resistors 25V ±1% ±200ppm/℃ 5.1kΩ 0201 Chip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, lib:R0201, F.Cu at (216.2, 66.5)
- added R3: 50mW Thick Film Resistors 25V ±5% ±200ppm/℃ 30kΩ 0201 Chip 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, lib:R0201, F.Cu at (180.3, 86.4)
- added R4: 50mW Thick Film Resistors 25V ±1% ±200ppm/℃ 10kΩ 0201 Chip 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, lib:R0201, F.Cu at (216.7, 54.1)
- added R5: 50mW Thick Film Resistors 25V ±1% ±200ppm/℃ 10kΩ 0201 Chip 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, lib:R0201, F.Cu at (216.7, 61.6)
- added R6: 50mW Thick Film Resistors 25V ±5% 0Ω 0201 Chip Resistor - S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, lib:R0201, F.Cu at (212.3, 61.6)
- added R7: 50mW Thick Film Resistors 25V ±1% ±200ppm/℃ 10kΩ 0201 Chip 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, lib:R0201, F.Cu at (184.8, 86.4)
- added R8: 50mW Thick Film Resistors 25V ±1% ±200ppm/℃ 10kΩ 0201 Chip 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, lib:R0201, F.Cu at (199.4, 61.7)
- added R9: 50mW Thick Film Resistors 25V ±1% ±200ppm/℃ 750Ω 0201 Chip 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, lib:R0201, F.Cu at (213.2, 84.5)
- added U1: ?, lib:QFN-24_L4.0-W4.0-P0.50-TL-EP2.7, F.Cu at (194.9, 84.6)
- added U2: ?, lib:VQFN-24_L4.0-W4.0-P0.50-TL-EP2.5, F.Cu at (195.2, 77.2)
- added U3: ?, lib:UQFN-10_L2.0-W1.5-P0.50-BL, F.Cu at (203.4, 77.1)
- added U4: ?, lib:CONN-TH_4P-XT30PW-M, F.Cu at (203.4, 103.8)
- added U5: ?, lib:USB-C_SMD-TYPE-C-31-M-12, F.Cu at (187.5, 102.1)
- added U6: ?, lib:USB-C_SMD-TYPE-C-31-M-12, F.Cu at (208.9, 118.0)
- added U7: ?, lib:DO-220AA_L3.4-W2.0-LS3.9-RD, F.Cu at (204.8, 67.4)
- added U8: ?, lib:IND-SMD_L5.2-W5.2_IHLP2020CZER2R2M11, F.Cu at (195.8, 69.0)
Other:
- board outline removed
