File: elec/layout/default/femtofox-mppt.kicad_pcb (KiCad board)
At the start: 2 copper layers, 33 parts, among them J1 ?, U1 ?, U2 ?, U3 ?, U4 ?, U5 ?, U6 ?, U7 ?, U8 ?

Commit message: eod 12/19/24
Parts:
- removed J1: ?, lib:CONN-SMD_4P-P1.00_SM04B-SRSS-TB-LF-SN
- removed R11, R12: 50mW Thick Film Resistors 25V ±1% ±200ppm/℃ 10kΩ 0201 Chip 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, lib:R0201
- removed U7: ?, lib:DO-220AA_L3.4-W2.0-LS3.9-RD
- removed U8: ?, lib:IND-SMD_L5.2-W5.2_IHLP2020CZER2R2M11
- R9: value 50mW Thick Film Resistors 25V ±1% ±200ppm/℃ 750Ω 0201 Chip Resistor - Surface Mount ROHS -> 50mW Thick Film Resistors 25V ±1% ±200ppm/℃ 10kΩ 0201 Chip Resistor - Surface Mount ROHS
- U1: footprint lib:QFN-24_L4.0-W4.0-P0.50-TL-EP2.7 -> lib:HDR-TH_11P-P2.54-V-M
- U2: footprint lib:VQFN-24_L4.0-W4.0-P0.50-TL-EP2.5 -> lib:HDR-TH_11P-P2.54-V-M
- U3: footprint lib:UQFN-10_L2.0-W1.5-P0.50-BL -> lib:QFN-24_L4.0-W4.0-P0.50-TL-EP2.7
- U4: footprint lib:CONN-TH_4P-XT30PW-M -> lib:VQFN-24_L4.0-W4.0-P0.50-TL-EP2.5
- U5: footprint lib:USB-C_SMD-TYPE-C-31-M-12 -> lib:DO-220AA_L3.4-W2.0-LS3.9-RD
- U6: footprint lib:USB-C_SMD-TYPE-C-31-M-12 -> lib:IND-SMD_L5.2-W5.2_IHLP2020CZER2R2M11
- moved U2 61.4 mm to (215.2, 135.2), turned to -90 degrees
- moved U1 50.7 mm to (197.5, 135.2), turned to -90 degrees
- moved R1 46.4 mm to (193.9, 90.7)
- moved C1 38.6 mm to (198.8, 86.5)
- moved R4 35.1 mm to (203.2, 86.5)
- moved U3 32.7 mm to (191.3, 107.5)
- moved U4 32.2 mm to (204.4, 136.0), turned to 180 degrees
- moved R5 30.1 mm to (207.7, 90.2)
- moved R6 30.1 mm to (203.2, 90.2)
- moved C12 29.3 mm to (188.7, 83.7)
- moved R10 29.0 mm to (207.7, 86.5)
- moved U5 28.0 mm to (189.7, 74.1), turned to 0 degrees
- moved C6 25.5 mm to (188.1, 91.9)
- moved R2 23.8 mm to (198.8, 82.8)
- moved R3 23.2 mm to (203.2, 82.8)
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Connections:
- R1 pad 2: p2 -> gnd
- R10 pad 1: dsel -> stat
- R10 pad 2: vcc-4 -> vcc-3
- R7 pad 1: scl -> ic-scl
- R8 pad 1: sda -> ic-sda
- R9 pad 1: p2 -> ce
- U1 pad 1: vcc-1 -> _5v
- U1 pad 10: ilim -> rx4
- U1 pad 11: ts -> tx4
- U1 pad 2: d_plus -> femtohat.row1-gnd
- U1 pad 3: d -> _3v3
- U1 pad 4: stat -> tx2
- U1 pad 5: scl -> rx2
- U1 pad 6: sda -> cs
- U1 pad 7: int -> sck
- U1 pad 8: otg -> mosi
- U1 pad 9: ce -> miso
- U2 pad 1: pa2 -> _1v8
- U2 pad 10: pb6 -> nrst
- U2 pad 11: pb5 -> nc
- U2 pad 2: extclk_slash_pa3 -> femtohat.row1-gnd
- U2 pad 3: uc-gnd -> _4c1
- U2 pad 4: vcc-3 -> _4c0
- U2 pad 5: pa4 -> _0a4
- U2 pad 6: pa5 -> irq
- U2 pad 7: pa6 -> busy
- U2 pad 8: pa7 -> femtohat.row2-scl
- U2 pad 9: pb7 -> femtohat.row2-sda
- U3 pad 1: d_plus -> vcc-1
- U3 pad 10: usb_sw.ic-vcc -> ilim
- U3 pad 2: d -> d_plus
- U3 pad 3: usb_sw.ic-dp -> d
- U3 pad 4: usb_sw.ic-dm -> stat
- U3 pad 5: usb_sw.ic-gnd -> ic-scl
- U3 pad 6: oe_hash -> ic-sda
- U3 pad 7: usb_sw.ic-dm-1 -> int
- U3 pad 8: usb_sw.ic-dp-1 -> otg
- U3 pad 9: dsel -> ce
- U4 pad 1: vcc-2 -> pa2
- U4 pad 2: gnd -> extclk_slash_pa3
- U4 pad 3: ts -> uc-gnd
- U4 pad 4: gnd -> vcc-3
- U5 pad 1: (no net) -> sw
- U5 pad 2: (no net) -> vcc-5
- U6 pad 1: (no net) -> sw
- U6 pad 2: (no net) -> vcc-3
